File: Electronics/v5/Display-2020/Display.kicad_pcb (KiCad board)
At the start: 4 copper layers, 104 x 40 mm, 120 parts, among them J1 Conn_02x07, T1 TouchPad, U2 APDS-9005

Commit message: Started work on v6 schematic
Routing:
- added copper zone on In2.Cu, net +5V
- added copper zone on In1.Cu, net GND
- removed copper zone on +5v, net +5V
- removed copper zone on GND, net GND
Other:
- net class Default removed
